Commit message: 修改部分限位，修改步态极性，配置自己的config和env

File: resources/robots/wrobot/urdf/wrobot_Fdd.urdf (robot description, URDF)
Before this commit: robot wrobot, 11 links, 10 joints
Links:
- link base_link: geometry collision box size=0.2 0.3 0.2; visual mesh filename=/data/resources/robots/wrobot/meshes/base_link.STL
- link left_ankle_link: geometry collision mesh filename=/data/resources/robots/wrobot/meshes/left_ankle_link.STL; visual mesh filename=/data/resources/robots/wrobot/meshes/left_ankle_link.STL
- link left_knee_link: geometry visual mesh filename=/data/resources/robots/wrobot/meshes/left_knee_link.STL
- link left_leg_pitch_link: geometry visual mesh filename=/data/resources/robots/wrobot/meshes/left_leg_pitch_link.STL
- link left_leg_roll_link: geometry visual mesh filename=/data/resources/robots/wrobot/meshes/left_leg_roll_link.STL
- link left_leg_yaw_link: geometry visual mesh filename=/data/resources/robots/wrobot/meshes/left_leg_yaw_link.STL
- link right_ankle_link: geometry collision mesh filename=/data/resources/robots/wrobot/meshes/right_ankle_link.STL; visual mesh filename=/data/resources/robots/wrobot/meshes/right_ankle_link.STL
- link right_knee_link: geometry visual mesh filename=/data/resources/robots/wrobot/meshes/right_knee_link.STL
- link right_leg_pitch_link: geometry visual mesh filename=/data/resources/robots/wrobot/meshes/right_leg_pitch_link.S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
- link right_leg_roll_link: geometry visual mesh filename=/data/resources/robots/wrobot/meshes/right_leg_roll_link.STL
- link right_leg_yaw_link: geometry visual mesh filename=/data/resources/robots/wrobot/meshes/right_leg_yaw_link.STL
