Commit message: 修改机器人碰撞模型

File: resources/robots/wrobot/urdf/wrobot.urdf (robot description, URDF)
Before this commit: robot wrobot, 11 links, 10 joints
Links:
- link base_link: geometry collision box size=0.2 0.3 0.2; visual mesh filename=package://wrobot/meshes/base_link.STL
- link left_knee_link: geometry visual mesh filename=package://wrobot/meshes/left_knee_link.STL
- link left_leg_pitch_link: geometry visual mesh filename=package://wrobot/meshes/left_leg_pitch_link.STL
- link left_leg_roll_link: geometry visual mesh filename=package://wrobot/meshes/left_leg_roll_link.STL
- link left_leg_yaw_link: geometry visual mesh filename=package://wrobot/meshes/left_leg_yaw_link.STL
- link right_knee_link: geometry visual mesh filename=package://wrobot/meshes/right_knee_link.STL
- link right_leg_pitch_link: geometry visual mesh filename=package://wrobot/meshes/right_leg_pitch_link.STL
- link right_leg_roll_link: geometry visual mesh filename=package://wrobot/meshes/right_leg_roll_link.STL
- link right_leg_yaw_link: geometry visual mesh filename=package://wrobot/meshes/right_leg_yaw_link.STL

Commit message: 修改目标高度，初始高度，urdf

File: resources/robots/wrobot/urdf/wrobot.urdf (robot description, URDF)
Before this commit: robot wrobot, 11 links, 10 joints
Links:
- link base_link: geometry collision box size=0.2 0.3 0.2; visual mesh filename=/home/wang/humanoid-gym/resources/robots/wrobot/meshes/base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
- link left_ankle_link: geometry collision mesh filename=/home/wang/humanoid-gym/resources/robots/wrobot/meshes/left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; visual mesh filename=/home/wang/humanoid-gym/resources/robots/wrobot/meshes/left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
- link left_knee_link: geometry visual mesh filename=/home/wang/humanoid-gym/resources/robots/wrobot/meshes/left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
- link left_leg_pitch_link: geometry visual mesh filename=/home/wang/humanoid-gym/resources/robots/wrobot/meshes/left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
- link left_leg_roll_link: geometry visual mesh filename=/home/wang/humanoid-gym/resources/robots/wrobot/meshes/left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
- link left_leg_yaw_link: geometry visual mesh filename=/home/wang/humanoid-gym/resources/robots/wrobot/meshes/left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
- link right_ankle_link: geometry collision mesh filename=/home/wang/humanoid-gym/resources/robots/wrobot/meshes/righ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; visual mesh filename=/home/wang/humanoid-gym/resources/robots/wrobot/meshes/righ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
- link right_knee_link: geometry visual mesh filename=/home/wang/humanoid-gym/resources/robots/wrobot/meshes/righ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
- link right_leg_pitch_link: geometry visual mesh filename=/home/wang/humanoid-gym/resources/robots/wrobot/meshes/righ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
- link right_leg_roll_link: geometry visual mesh filename=/home/wang/humanoid-gym/resources/robots/wrobot/meshes/righ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
- link right_leg_yaw_link: geometry visual mesh filename=/home/wang/humanoid-gym/resources/robots/wrobot/meshes/righ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

Commit message: 修改pd参数，修改urdf的limit

File: resources/robots/wrobot/urdf/wrobot.urdf (robot description, URDF)
Before this commit: robot wrobot, 11 links, 10 joints
Joints:
- joint left_ankle_joint: limit lower=-1.3 upper=1.3 effort=100 velocity=12 -> lower=-1.3 upper=1.3 effort=25 velocity=12
- joint left_knee_joint: limit lower=0 upper=2.2 effort=250 velocity=12 -> lower=0 upper=2.2 effort=70 velocity=12
- joint left_leg_pitch_joint: limit lower=-1.75 upper=0.17 effort=250 velocity=12 -> lower=-1.75 upper=0.17 effort=70 velocity=12
- joint left_leg_roll_joint: limit lower=-0.14 upper=0.2 effort=100 velocity=12 -> lower=-0.14 upper=0.2 effort=25 velocity=12
- joint left_leg_yaw_joint: limit lower=-0.3 upper=0.16 effort=100 velocity=12 -> lower=-0.3 upper=0.16 effort=25 velocity=12
- joint right_ankle_joint: limit lower=-1.3 upper=1.3 effort=100 velocity=12 -> lower=-1.3 upper=1.3 effort=25 velocity=12
- joint right_knee_joint: limit lower=0 upper=2.2 effort=250 velocity=12 -> lower=0 upper=2.2 effort=70 velocity=12
- joint right_leg_pitch_joint: limit lower=-1.75 upper=0.17 effort=250 velocity=12 -> lower=-1.75 upper=0.17 effort=70 velocity=12
- joint right_leg_roll_joint: limit lower=-0.2 upper=0.14 effort=100 velocity=12 -> lower=-0.2 upper=0.14 effort=25 velocity=12
- joint right_leg_yaw_joint: limit lower=-0.16 upper=0.3 effort=100 velocity=12 -> lower=-0.16 upper=0.3 effort=25 velocity=12

Commit message: 修改pd，max_torque

File: resources/robots/wrobot/urdf/wrobot.urdf (robot description, URDF)
Before this commit: robot wrobot, 11 links, 10 joints
Joints:
- joint left_ankle_joint: limit lower=-1.3 upper=1.3 effort=25 velocity=12 -> lower=-1.3 upper=1.3 effort=50 velocity=12
- joint left_knee_joint: limit lower=0 upper=2.2 effort=70 velocity=12 -> lower=0 upper=2.2 effort=140 velocity=12
- joint left_leg_pitch_joint: limit lower=-1.75 upper=0.17 effort=70 velocity=12 -> lower=-1.75 upper=0.17 effort=140 velocity=12
- joint left_leg_roll_joint: limit lower=-0.14 upper=0.2 effort=25 velocity=12 -> lower=-0.14 upper=0.2 effort=50 velocity=12
- joint left_leg_yaw_joint: limit lower=-0.3 upper=0.16 effort=25 velocity=12 -> lower=-0.3 upper=0.16 effort=50 velocity=12
- joint right_ankle_joint: limit lower=-1.3 upper=1.3 effort=25 velocity=12 -> lower=-1.3 upper=1.3 effort=50 velocity=12
- joint right_knee_joint: limit lower=0 upper=2.2 effort=70 velocity=12 -> lower=0 upper=2.2 effort=140 velocity=12
- joint right_leg_pitch_joint: limit lower=-1.75 upper=0.17 effort=70 velocity=12 -> lower=-1.75 upper=0.17 effort=140 velocity=12
- joint right_leg_roll_joint: limit lower=-0.2 upper=0.14 effort=25 velocity=12 -> lower=-0.2 upper=0.14 effort=50 velocity=12
- joint right_leg_yaw_joint: limit lower=-0.16 upper=0.3 effort=25 velocity=12 -> lower=-0.16 upper=0.3 effort=50 velocity=12

Commit message: v8_change_pd_limit_torque

File: resources/robots/wrobot/urdf/wrobot.urdf (robot description, URDF)
Before this commit: robot wrobot, 11 links, 10 joints
Joints:
- joint left_ankle_joint: limit lower=-1.3 upper=1.3 effort=50 velocity=12 -> lower=-1.3 upper=1.3 effort=70 velocity=12
- joint left_knee_joint: limit lower=0 upper=2.2 effort=140 velocity=12 -> lower=0 upper=2.2 effort=200 velocity=12
- joint left_leg_pitch_joint: limit lower=-1.75 upper=0.17 effort=140 velocity=12 -> lower=-1.75 upper=0.17 effort=200 velocity=12
- joint left_leg_roll_joint: limit lower=-0.14 upper=0.2 effort=50 velocity=12 -> lower=-0.14 upper=0.2 effort=70 velocity=12
- joint left_leg_yaw_joint: limit lower=-0.3 upper=0.16 effort=50 velocity=12 -> lower=-0.3 upper=0.16 effort=70 velocity=12
- joint right_ankle_joint: limit lower=-1.3 upper=1.3 effort=50 velocity=12 -> lower=-1.3 upper=1.3 effort=70 velocity=12
- joint right_knee_joint: limit lower=0 upper=2.2 effort=140 velocity=12 -> lower=0 upper=2.2 effort=200 velocity=12
- joint right_leg_pitch_joint: limit lower=-1.75 upper=0.17 effort=140 velocity=12 -> lower=-1.75 upper=0.17 effort=200 velocity=12
- joint right_leg_roll_joint: limit lower=-0.2 upper=0.14 effort=50 velocity=12 -> lower=-0.2 upper=0.14 effort=70 velocity=12
- joint right_leg_yaw_joint: limit lower=-0.16 upper=0.3 effort=50 velocity=12 -> lower=-0.16 upper=0.3 effort=70 velocity=12
